File: hardware/keyboard.kicad_pcb (KiCad board)
At the start: 2 copper layers, 305.7 x 121 mm, 175 parts, among them J1 Conn_02x20_Odd_Even, J2 USB_C_Receptacle_16P

Commit message: feat(hardware): update kbd layout
Parts:
- moved SW-80 19.1 mm to (358.7, 72.4)
- moved SW-74 19.1 mm to (339.6, 72.3)
Connections:
- D3 pad 2: /L1 -> (no net)
- D4 pad 2: /L2 -> (no net)
- D5 pad 2: /L3 -> (no net)
- J1 pad 2: /L3 -> VDD33
- J1 pad 4: /L2 -> VDD33
- J1 pad 6: /L1 -> VDD33
- J1 pad 8: (no net) -> VDD33
